File: escPCB.kicad_sch (KiCad schematic)
At the start: 57 parts, among them IC1 W25Q16JVSNIQ, J1 Terminal, J2 2137160001, Q1 BC857, Q10 BC857, Q11 BC857, Q12 BC857, Q13 BC847, Q14 BC847, Q15 BC847, Q2 BC857, Q3 BC857, Q4 BC847, Q5 BC847, Q6 BC847, Q7 BC847, Q8 BC847, Q9 BC847, U1 RP2040, U2 LD1117S33TR_SOT223, X1 ABM8-272-T3

Commit message: schematic v2 with some footprints
Parts:
- added C13, C14: 100n, Capacitor_SMD:C_0805_2012Metric, symbol Device:C
- added C15: 1u, Capacitor_SMD:C_0805_2012Metric, symbol Device:C
- added J3: XT60-M, SPROGEE3:AMASS_XT60-M, symbol XT60-M:XT60-M
- added J4, J5: Conn_01x03_Pin, Connector_JST:JST_PH_S3B-PH-K_1x03_P2.00mm_Horizontal, symbol Connector:Conn_01x03_Pin
- added J6: Conn_01x02_Pin, Connector_JST:JST_PH_S2B-PH-K_1x02_P2.00mm_Horizontal, symbol Connector:Conn_01x02_Pin
- added JP1, JP2: SolderJumper_2_Open, Jumper:SolderJumper-2_P1.3mm_Open_RoundedPad1.0x1.5mm, symbol Jumper:SolderJumper_2_Open
- added JP3: SolderJumper_3_Open, Jumper:SolderJumper-3_P1.3mm_Bridged2Bar12_Pad1.0x1.5mm_NumberLabels, symbol Jumper:SolderJumper_3_Open
- added R19, R20: 27, Resistor_SMD:R_0805_2012Metric, symbol Device:R
- AH1: renamed from AH; footprint (none) -> SPROGEE3:IPD70P04P4L08ATMA2
- AL1: renamed from AL; footprint (none) -> SPROGEE3:IPD70P04P4L08ATMA2
- BH1: renamed from BH; footprint (none) -> SPROGEE3:IPD70P04P4L08ATMA2
- BL1: renamed from BL; footprint (none) -> SPROGEE3:IPD70P04P4L08ATMA2
- C1, C10, C11, C12, C2, C3, C4, C5, C6, C7, C8, C9: footprint (none) -> Capacitor_SMD:C_0805_2012Metric
- CH1: renamed from CH; footprint (none) -> SPROGEE3:IPD70P04P4L08ATMA2
- CL1: renamed from CL; footprint (none) -> SPROGEE3:IPD70P04P4L08ATMA2
- IC1: footprint (none) -> SPROGEE3:W25Q
- J2: footprint 2137160001:MOLEX_2137160001 -> SPROGEE3:MOLEX_2137160001 USB-C
- R1, R16, R17, R18, R2, R3, R4, R5, R6, R7, R8, R9: footprint (none) -> Resistor_SMD:R_0805_2012Metric
- R10, R11, R12, R13, R14, R15: value R -> 1k; footprint (none) -> Resistor_SMD:R_0805_2012Metric
- X1: footprint ABM8-272-T3_ABR -> Library:ABM8-272-T3_ABR
Connections:
- net +3.3V: now also JP3.3 (B); no longer C5.1, U2.2 (VO)
- net +BATT: now also J3.P (POS), JP2.2 (B); no longer C4.1, U2.3 (VI)
- net -BATT: no longer AL1.3 (S), BL1.3 (S), C1.2, C10.2, C11.2, C12.2, C2.2, C3.2, C4.2, C5.2, C6.2, C7.2, C8.2, C9.2, CL1.3 (S), IC1.4 (GND), J2.A1 (GND1), J2.A12 (GND2), J2.B1 (GND3), J2.B12 (GND4), J2.SH1 (SHIELD1), J2.SH2 (SHIELD2), J2.SH3 (SHIELD3), J2.SH4 (SHIELD4), Q1.3 (C), Q2.3 (C), Q3.3 (C), Q7.2 (E), Q8.2 (E), Q9.2 (E), R10.2, R11.2, R12.2, R17.1, R18.1, U1.19 (TESTEN), U1.57 (GND), U2.1 (GND), X1.2, X1.4
- net USB_D+: now also R19.1; no longer U1.47 (USB_DP)
- net USB_D-: now also R20.1; no longer U1.46 (USB_DM)
- net +1V1: now reaches U1.23 (DVDD), U1.50 (DVDD)
- net +1V1: now also U1.45 (VREG_VOUT), C13.1, C14.1, C15.1
- net SWCLK: now reaches U1.24 (SWCLK)
- net SWCLK: now also J5.1 (Pin_1)
- net SWD: now reaches U1.25 (SWD)
- net SWD: now also J5.2 (Pin_2)
- net RP_UART_TX: now reaches U1.27 (GPIO16)
- net RP_UART_TX: now also J4.1 (Pin_1)
- net RP_UART_RX: now reaches U1.28 (GPIO17)
- net RP_UART_RX: now also J4.2 (Pin_2)
- new net: C4.1, JP2.1 (A), U2.3 (VI)
- new net: C4.2, C5.2, JP1.2 (B), U2.1 (GND)
- new net: R19.2, U1.47 (USB_DP)
- new net: C5.1, JP3.1 (A), U2.2 (VO)
- new net: J6.1 (Pin_1), JP3.2 (C)
- new net: R20.2, U1.46 (USB_DM)
- new net GND: AL1.3 (S), BL1.3 (S), C1.2, C10.2, C11.2, C12.2, C13.2, C14.2, C15.2, C2.2, C3.2, C6.2, C7.2, C8.2, C9.2, CL1.3 (S), IC1.4 (GND), J2.A1 (GND1), J2.A12 (GND2), J2.B1 (GND3), J2.B12 (GND4), J2.SH1 (SHIELD1), J2.SH2 (SHIELD2), J2.SH3 (SHIELD3), J2.SH4 (SHIELD4), J3.N (NEG), J4.3 (Pin_3), J5.3 (Pin_3), J6.2 (Pin_2), JP1.1 (A), Q1.3 (C), Q2.3 (C), Q3.3 (C), Q7.2 (E), Q8.2 (E), Q9.2 (E), R10.2, R11.2, R12.2, R17.1, R18.1, U1.19 (TESTEN), U1.57 (GND), X1.2, X1.4
- no-connect marks 34 -> 31
Other:
- note added: "3V3 Terminal"
- note added: "Battery Terminal"
- note added: "Motor Sensing Circuit Here!"
- note added: "SWDIO Connector"
- note added: "UART Connector"
- moved on the sheet: C1, C10, C11, C12, C2, C3, C4, C5, C9, Q10, Q11, Q12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

Commit message: v3 PCB design from Desktop
Had to upload differently cause it was made on my desktop
Parts:
- added C16: C, Capacitor_SMD:C_0805_2012Metric, symbol Device:C
- added CR1: LM211N, SPROGEE3:DIP-8_STM, symbol LM211N Comparator:LM211N
- added H1, H2, H3, H4: MountingHole, MountingHole:MountingHole_3.2mm_M3, symbol Mechanical:MountingHole
- added R21, R22, R23, R24: 33k, Resistor_SMD:R_0805_2012Metric, symbol Device:R
- added R25, R27: 1k, Resistor_SMD:R_0805_2012Metric, symbol Device:R
- added R26: 10k, Resistor_SMD:R_0805_2012Metric, symbol Device:R
- added S1, S2: 431183015816, SPROGEE3:431183015816, symbol 431183015816:431183015816
- AL1, BL1, CL1: footprint SPROGEE3:IPD70P04P4L08ATMA2 -> SPROGEE3:IPB70N12S311ATMA1
- X1: footprint Library:ABM8-272-T3_ABR -> SPROGEE3:ABM8-272-T3_ABR
Connections:
- net +3.3V: now also JP3.2 (C), U1.44 (VREG_IN), R25.2, R26.1; no longer JP3.3 (B)
- net +BATT: now also CR1.8 (VCC+)
- net GND: now also C16.2, CR1.1 (GROUND), CR1.4 (VCC-), S1.1, S1.3, S1.GND1, S1.GND2, S2.1, S2.3, S2.GND1, S2.GND2
- net QSPI_SS: now also R27.2
- net L1: now reaches AH1.2 (S), AL1.2 (D), J1.1 (Pin_1)
- net L1: now also R21.2, R24.1
- net L2: now reaches BH1.2 (S), BL1.2 (D), J1.2 (Pin_2)
- net L2: now also R22.2
- net L3: now reaches CH1.2 (S), CL1.2 (D), J1.3 (Pin_3)
- net L3: now also R23.2
- net at J6.1 (Pin_1): now also JP3.3 (B); no longer JP3.2 (C)
- net at U1.26 (RUN): now also R26.2, S1.2, S1.4
- net PHASED: now reaches U1.38 (GPIO26_ADC0)
- net PHASED: now also C16.1, CR1.7 (OUTPUT), R25.1
- new net: R27.1, S2.2, S2.4
- new net: CR1.2 (NONINVERTINGINPUT), R24.2
- new net: CR1.3 (INVERTINGINPUT), R21.1, R22.1, R23.1
Other:
- note removed: "Motor Sensing Circuit Here!"
- moved on the sheet: C12, C13, C14, C15, C6, IC1
