File: escPCB.kicad_pcb (KiCad board)
At the start: 2 copper layers, 60 x 100 mm, 88 parts, among them IC1 W25Q16JVSNIQ, J1 Terminal, J2 2137160001, J3 XT60-M, J4 Conn_01x03_Pin, J5 Conn_01x03_Pin, J6 Conn_01x02_Pin, Q1 BC857, Q10 BC857, Q11 BC857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

Commit message: with 3d print casing
Parts:
- C16: value C -> 10n
Changed lines of the file:
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@@
 			)
 		)
-		(property "Value" "C"
+		(property "Value" "10n"
 			(at 0 1.68 90)
 			(layer "F.Fab")
